File: nrf24.kicad_pcb (KiCad board)
At the start: 2 copper layers, 0 parts

Commit message: Initial layout
Parts:
- added J1: Conn_01x08, Pin_Headers:Pin_Header_Straight_1x08_Pitch2.54mm, F.Cu at (155.9, 110.0)
- added U1: nRF24, nrf_footprints:nrf24_footprint, F.Cu at (137.2, 119.4)
Routing:
- net Net-(J1-Pad1): track 0.00 -> 27.0 mm
- net Net-(J1-Pad2): track 0.00 -> 24.4 mm
- net Net-(J1-Pad5): track 0.00 -> 22.9 mm
- net Net-(J1-Pad8): track 0.00 -> 15.5 mm
- net Net-(J1-Pad7): track 0.00 -> 15.3 mm
- net Net-(J1-Pad3): track 0.00 -> 15.2 mm
- net Net-(J1-Pad6): track 0.00 -> 14.3 mm
- net Net-(J1-Pad4): track 0.00 -> 11.2 mm
Other:
- board outline added: 33 x 24 mm
- net class Default: clearance 0.2 -> 0.1524; trace_width 0.25 -> 0.3048; via_dia 0.6 -> 0.508; via_drill 0.4 -> 0.3302
- rule trace_clearance: 0.2 -> 0.1524
- board text added: "CE"
- board text added: "CSN"
- board text added: "GND"
- board text added: "IRQ"
- board text added: "MISO"
- board text added: "MOSI"
- board text added: "SCK"
- board text added: "V1.0"
- board text added: "Vcc"

Commit message: final layout and gerber files
Parts:
- added C1: 10uF, Capacitors_THT:CP_Radial_D10.0mm_P5.00mm, F.Cu at (141.2, 130.2)
Routing:
- net Net-(C1-Pad2): track 27.0 -> 44.6 mm
- net Net-(C1-Pad1): track 15.5 -> 25.4 mm
- added copper zone on F.Cu, net Net-(C1-Pad2)
Other:
- board size 33 x 24 mm -> 33 x 32.6 mm
- rule trace_min: 0.2 -> 0.1524
- rule via_min_drill: 0.3 -> 0.3302
- rule via_min_size: 0.4 -> 0.4826
- board text added: "nRF24 Breakout Board"
